File: LPF Relay Control1.kicad_sch (KiCad schematic)
At the start: 24 parts, among them K1 EA2-5NU, K2 EA2-5NU, K3 EA2-5NU, K4 EA2-5NU, K5 EA2-5NU, K6 EA2-5NU, K7 EA2-5NU, K8 EA2-5NU, Q1 BSS123, Q3 BSS123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

Commit message: Working on LPF control and actual filters.  They are intertwingled pretty tightly.  Also ran ERC and beat out some errors.
Connections:
- net GND: now also K1.9 (N.C._2)
- net LPF0-OUT: now reaches K2.8 (COM_2)
- net LPF0-IN: now reaches K1.8 (COM_2)
- net LPF0 renamed LPF0-CTL
- net LPF1 renamed LPF1-CTL
- net LPF2 renamed LPF2-CTL
- net LPF3 renamed LPF3-CTL
- no-connect marks 0 -> 19
Other:
- added sheet LPF0 (LPF0.kicad_sch)

Commit message: moved LPF0 to LPF as I can fit them all into one schematic
Other:
- sheet LPF0 renamed LPF
- sheet LPF: file LPF0.kicad_sch -> LPF.kicad_sch
Changed lines of the file:
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@@
 			(color 0 0 0 0.0000)
 		)
-		(property "Sheetname" "LPF0"
+		(property "Sheetname" "LPF"
 			(at 29.21 33.5784 0)
 			(effects
@@
 			)
 		)
-		(property "Sheetfile" "LPF0.kicad_sch"
+		(property "Sheetfile" "LPF.kicad_sch"
 			(at 29.21 47.5746 0)
 			(effects

Commit message: placed LPF chains in sub-schematic.  ERC passes
Connections:
- net GND: now also K3.9 (N.C._2)
- net LPF1-OUT: now reaches K4.8 (COM_2)
- net LPF2-IN: now reaches K5.8 (COM_2)
- net LPF2-OUT: now reaches K6.8 (COM_2)
- net LPF3-IN: now reaches K7.8 (COM_2)
- net LPF1-IN: now reaches K3.8 (COM_2)
- net LPF3-OUT: now reaches K8.8 (COM_2)
- no-connect marks 19 -> 22
Other:
- sheet LPF ports: added LPF1-IN, LPF1-OUT, LPF2-IN, LPF2-OUT, LPF3-IN, LPF3-OUT; removed none

Commit message: checkpoint progress, working on LPF chains
Connections:
- no-connect marks 22 -> 40
Changed lines of the file:
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@@
+	)
+	(no_connect
+		(at 162.56 107.95)
 	)
 	(no_connect
@@
 	(no_connect
 		(at 106.68 67.31)
+	)
+	(no_connect
+		(at 177.8 74.93)
+	)
+	(no_connect
+		(at 177.8 113.03)
+	)
+	(no_connect
+		(at 177.8 107.95)
 	)
 	(no_connect
@@
 	)
 	(no_connect
+		(at 177.8 36.83)
+	)
+	(no_connect
 		(at 162.56 74.93)
+	)
+	(no_connect
+		(at 177.8 72.39)
+	)
+	(no_connect
+		(at 177.8 34.29)
 	)
 	(no_connect
@@
 	)
 	(no_connect
+		(at 177.8 110.49)
+	)
+	(no_connect
+		(at 162.56 148.59)
+	)
+	(no_connect
 		(at 233.68 39.37)
+	)
+	(no_connect
+		(at 177.8 31.75)
 	)
 	(no_connect
@@
 	)
 	(no_connect
+		(at 177.8 69.85)
+	)
+	(no_connect
+		(at 162.56 110.49)
+	)
+	(no_connect
+		(at 162.56 146.05)
+	)
+	(no_connect
+		(at 177.8 151.13)
+	)
+	(no_connect
 		(at 177.8 153.67)
 	)
@@
 	)
 	(no_connect
+		(at 177.8 146.05)
+	)
+	(no_connect
+		(at 177.8 148.59)
+	)
+	(no_connect
+		(at 162.56 151.13)
+	)
+	(no_connect
 		(at 162.56 105.41)
 	)
 	(no_connect
+		(at 162.56 113.03)
+	)
+	(no_connect

Commit message: fleshed out LPF chains.  ERC passes
Other:
- sheet LPF renamed LPF Chain
Changed lines of the file:
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@@
 			(color 0 0 0 0.0000)
 		)
-		(property "Sheetname" "LPF"
+		(property "Sheetname" "LPF Chain"
 			(at 29.21 33.5784 0)
 			(effects

Commit message: added RF through LPF chains
Connections:
- net RF-OUT: now reaches K4.7 (N.O._2)
- net RF-OUT: now also K2.7 (N.O._2), K6.7 (N.O._2), K8.7 (N.O._2)
- net RF-IN: now reaches K5.7 (N.O._2)
- net RF-IN: now also K1.7 (N.O._2), K3.7 (N.O._2), K7.7 (N.O._2)
Changed lines of the file:
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@@
 	(title_block
 		(title "QMX Amp")
-		(date "2024-08-08")
+		(date "2024-08-09")
 		(rev "v0.1")
 		(company "WA7GIL")
@@
 	(wire
 		(pts
-			(xy 102.87 34.29) (xy 106.68 34.29)
+			(xy 97.79 34.29) (xy 106.68 34.29)
 		)
 		(stroke
@@
 	(wire
 		(pts
-			(xy 102.87 72.39) (xy 106.68 72.39)
+			(xy 97.79 72.39) (xy 106.68 72.39)
 		)
 		(stroke
@@
 	(wire
 		(pts
-			(xy 102.87 110.49) (xy 106.68 110.49)
+			(xy 97.79 110.49) (xy 106.68 110.49)
 		)
 		(stroke
@@
 	(wire
 		(pts
-			(xy 102.87 148.59) (xy 106.68 148.59)
+			(xy 97.79 148.59) (xy 106.68 148.59)
 		)
 		(stroke
@@
 	)
 	(label "LPF3-IN"
-		(at 102.87 148.59 180)
+		(at 97.79 148.59 180)
 		(fields_autoplaced yes)
 		(effects
@@
 	)
 	(label "LPF1-IN"
-		(at 102.87 72.39 180)
+		(at 97.79 72.39 180)
 		(fields_autoplaced yes)
 		(effects
@@
 	)
 	(label "LPF0-IN"
-		(at 102.87 34.29 180)
+		(at 97.79 34.29 180)
 		(fields_autoplaced yes)
 		(effects
@@
 	)
 	(label "LPF2-IN"
-		(at 102.87 110.49 180)
+		(at 97.79 110.49 180)
 		(fields_autoplaced yes)
 		(effects
@@
 		)
 	)
+	(global_label "RF-OUT"
+		(shape bidirectional)
+		(at 233.68 151.13 0)
+		(fields_autoplaced yes)
+		(effects
+			(font
+				(size 1.27 1.27)
+			)
+			(justify left)
+		)
+		(property "Intersheetrefs" "${INTERSHEET_REFS}"
+			(at 245.3359 151.13 0)
+			(effects
+				(font
+					(size 1.27 1.27)
+				)
+				(justify left)
+				(hide yes)
+			)
+		)
+	)
+	(global_label "RF-IN"
+		(shape bidirectional)
+		(at 106.68 146.05 180)
+		(fields_autoplaced yes)
+		(effects
+			(font
+				(size 1.27 1.27)
+			)
+			(justify right)
+		)
+		(property "Intersheetrefs" "${INTERSHEET_REFS}"
+			(at 96.7174 146.05 0)
+			(effects
+				(font
+					(size 1.27 1.27)
+				)
+				(justify right)
+				(hide yes)
+			)
+		)
+	)
+	(global_label "RF-IN"
+		(shape bidirectional)
+		(at 106.68 107.95 180)
+		(fields_autoplaced yes)
+		(effects
+			(font
+				(size 1.27 1.27)
+			)
+			(justify right)
+		)
+		(property "Intersheetrefs" "${INTERSHEET_REFS}"
+			(at 96.7174 107.95 0)
+			(effects
+				(font
+					(size 1.27 1.27)
+				)
+				(justify right)
+				(hide yes)
+			)
+		)
+	)
+	(global_label "RF-OUT"
+		(shape bidirectional)
+		(at 233.68 74.93 0)
+		(fields_autoplaced yes)
+		(effects
+			(font
+				(size 1.27 1.27)
+			)
+			(justify left)
+		)
+		(property "Intersheetrefs" "${INTERSHEET_REFS}"
+			(at 245.3359 74.93 0)
+			(effects
+				(font
+					(size 1.27 1.27)
+				)
+				(justify left)
+				(hide yes)
+			)
+		)
+	)
+	(global_label "RF-IN"
+		(shape bidirectional)
+		(at 106.68 69.85 180)
+		(fields_autoplaced yes)
+		(effects
+			(font
+				(size 1.27 1.27)
+			)
+			(justify right)
+		)
+		(property "Intersheetrefs" "${INTERSHEET_REFS}"
+			(at 96.7174 69.85 0)
+			(effects
+				(font
+					(size 1.27 1.27)
+				)
+				(justify right)
+				(hide yes)
+			)
+		)
+	)
+	(global_label "RF-IN"
+		(shape bidirectional)
+		(at 106.68 31.75 180)
+		(fields_autoplaced yes)
+		(effects
+			(font
+				(size 1.27 1.27)
+			)
+			(justify right)
+		)
+		(property "Intersheetrefs" "${INTERSHEET_REFS}"
+			(at 96.7174 31.75 0)
+			(effects
+				(font
+					(size 1.27 1.27)
+				)
+				(justify right)
+				(hide yes)
+			)
+		)
+	)
+	(global_label "RF-OUT"
+		(shape bidirectional)
+		(at 233.68 113.03 0)
+		(fields_autoplaced yes)
+		(effects
+			(font
+				(size 1.27 1.27)
+			)
+			(justify left)
+		)
+		(property "Intersheetrefs" "${INTERSHEET_REFS}"
+			(at 245.3359 113.03 0)
+			(effects
+				(font
+					(size 1.27 1.27)
+				)
+				(justify left)
+				(hide yes)
+			)
+		)
+	)
+	(global_label "RF-OUT"
+		(shape bidirectional)
+		(at 233.68 36.83 0)
+		(fields_autoplaced yes)
+		(effects
+			(font
+				(size 1.27 1.27)
+			)
+			(justify left)
+		)
+		(property "Intersheetrefs" "${INTERSHEET_REFS}"
+			(at 245.3359 36.83 0)
+			(effects
+				(font
+					(size 1.27 1.27)
+				)
+				(justify left)
+				(hide yes)
+			)
+		)
+	)

Commit message: worked on strange stuff on btm of LPF filter chain schematic.  ERC passes
Connections:
- net RF-IN renamed RF-IN-PAST-SW
Changed lines of the file:
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@@
 	)
 	(label "LPF3-IN"
-		(at 97.79 148.59 180)
+		(at 97.79 148.59 270)
 		(fields_autoplaced yes)
 		(effects
@@
 	)
 	(label "LPF1-IN"
-		(at 97.79 72.39 180)
+		(at 97.79 72.39 270)
 		(fields_autoplaced yes)
 		(effects
@@
 	)
 	(label "LPF0-IN"
-		(at 97.79 34.29 180)
+		(at 97.79 34.29 270)
 		(fields_autoplaced yes)
 		(effects
@@
 	)
 	(label "LPF2-IN"
-		(at 97.79 110.49 180)
+		(at 97.79 110.49 270)
 		(fields_autoplaced yes)
 		(effects
@@
 		)
 	)
-	(global_label "RF-IN"
+	(global_label "RF-IN-PAST-SW"
 		(shape bidirectional)
 		(at 106.68 146.05 180)
@@
 		)
 		(property "Intersheetrefs" "${INTERSHEET_REFS}"
-			(at 96.7174 146.05 0)
+			(at 86.376 146.05 0)
 			(effects
 				(font
@@
 		)
 	)
-	(global_label "RF-IN"
+	(global_label "RF-IN-PAST-SW"
 		(shape bidirectional)
 		(at 106.68 107.95 180)
@@
 		)
 		(property "Intersheetrefs" "${INTERSHEET_REFS}"
-			(at 96.7174 107.95 0)
+			(at 86.376 107.95 0)
 			(effects
 				(font
@@
 		)
 	)
-	(global_label "RF-IN"
+	(global_label "RF-IN-PAST-SW"
 		(shape bidirectional)
 		(at 106.68 69.85 180)
@@
 		)
 		(property "Intersheetrefs" "${INTERSHEET_REFS}"
-			(at 96.7174 69.85 0)
+			(at 86.376 69.85 0)
 			(effects
 				(font
@@
 		)
 	)
-	(global_label "RF-IN"
+	(global_label "RF-IN-PAST-SW"
 		(shape bidirectional)
 		(at 106.68 31.75 180)
@@
 		)
 		(property "Intersheetrefs" "${INTERSHEET_REFS}"
-			(at 96.7174 31.75 0)
-			(effects
-				(font
+			(at 86.376 31.75 0)
+			(effects
+				(font
