File: LPF Relay Control1.kicad_sch (KiCad schematic)
At the start: 24 parts, among them K1 EA2-5NU, K2 EA2-5NU, K3 EA2-5NU, K4 EA2-5NU, K5 EA2-5NU, K6 EA2-5NU, K7 EA2-5NU, K8 EA2-5NU, Q1 BSS123, Q3 BSS123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

Commit message: RF-IN-PAST-SW now RF-INTO-FILTERS
Connections:
- net RF-IN-PAST-SW renamed RF-INTO-FILTERS
Changed lines of the file:
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@@
 		)
 	)
-	(global_label "RF-IN-PAST-SW"
+	(global_label "RF-INTO-FILTERS"
 		(shape bidirectional)
 		(at 106.68 146.05 180)
@@
 		)
 		(property "Intersheetrefs" "${INTERSHEET_REFS}"
-			(at 86.376 146.05 0)
+			(at 85.5293 146.05 0)
 			(effects
 				(font
@@
 		)
 	)
-	(global_label "RF-IN-PAST-SW"
+	(global_label "RF-INTO-FILTERS"
 		(shape bidirectional)
 		(at 106.68 107.95 180)
@@
 		)
 		(property "Intersheetrefs" "${INTERSHEET_REFS}"
-			(at 86.376 107.95 0)
+			(at 85.5293 107.95 0)
 			(effects
 				(font
@@
 		)
 	)
-	(global_label "RF-IN-PAST-SW"
+	(global_label "RF-INTO-FILTERS"
 		(shape bidirectional)
 		(at 106.68 69.85 180)
@@
 		)
 		(property "Intersheetrefs" "${INTERSHEET_REFS}"
-			(at 86.376 69.85 0)
+			(at 85.5293 69.85 0)
 			(effects
 				(font
@@
 		)
 	)
-	(global_label "RF-IN-PAST-SW"
+	(global_label "RF-INTO-FILTERS"
 		(shape bidirectional)
 		(at 106.68 31.75 180)
@@
 		)
 		(property "Intersheetrefs" "${INTERSHEET_REFS}"
-			(at 86.376 31.75 0)
+			(at 85.5293 31.75 0)
 			(effects
 				(font

Commit message: +5V REG now connected to all LPF relay coils
Connections:
- net +5V renamed +5V REG
Changed lines of the file:
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@@
+		)
+	)
+	(global_label "+5V REG"
+		(shape bidirectional)
+		(at 170.18 19.05 180)
+		(fields_autoplaced yes)
+		(effects
+			(font
+				(size 1.27 1.27)
+			)
+			(justify right)
+		)
+		(property "Intersheetrefs" "${INTERSHEET_REFS}"
+			(at 157.5566 19.05 0)
+			(effects
+				(font
+					(size 1.27 1.27)
+				)
+				(justify right)
+				(hide yes)
+			)
 		)
 	)
@@
 					(unit 1)
 				)
-			)
-		)
-	)
-	(symbol
-		(lib_id "power:+5V")
-		(at 170.18 19.05 0)
-		(unit 1)
-		(exclude_from_sim no)
-		(in_bom yes)
-		(on_board yes)
-		(dnp no)
-		(fields_autoplaced yes)
-		(property "Reference" "#PWR03"
-			(at 170.18 22.86 0)
-			(effects
-				(font
-					(size 1.27 1.27)
-				)
-				(hide yes)
-			)
-		)
-		(property "Value" "+5V"
-			(at 170.18 13.97 0)
-			(effects
-				(font
-					(size 1.27 1.27)
-				)
-			)
-		)
-		(property "Footprint" ""
-			(at 170.18 19.05 0)
-			(effects
-				(font
-					(size 1.27 1.27)
-				)
-				(hide yes)
-			)
-		)
-		(property "Datasheet" ""
-			(at 170.18 19.05 0)
-			(effects
-				(font
-					(size 1.27 1.27)
-				)
-				(hide yes)
-			)
-		)
-		(property "Description" "Power symbol creates a global label with name \"+5V\""
-			(at 170.18 19.05 0)
-			(effects
-				(font
-					(size 1.27 1.27)
-				)
-				(hide yes)
-			)
-		)
-		(pin "1"
-		)
-		(instances
-			(project "QMX-amp"
-				(path "/e63e39d7-6ac0-4ffd-8aa3-1841a4541b55/a2d04ef4-5ee1-49c1-8112-2f230613295c"
-					(reference "#PWR03")
-					(unit 1)
-				)

Commit message: trying to get K1 & K2 appear in multiple places, yet be recognized as identical.  Currently reporting dup K1
Parts:
- renumbered K2 to K10, K1 to K9
Changed lines of the file:
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@@
 		(on_board yes)
 		(dnp no)
-		(property "Reference" "K2"
+		(property "Reference" "K10"
 			(at 206.502 29.21 0)
 			(effects
@@
 			(project "QMX-amp"
 				(path "/e63e39d7-6ac0-4ffd-8aa3-1841a4541b55/a2d04ef4-5ee1-49c1-8112-2f230613295c"
-					(reference "K2")
+					(reference "K10")
 					(unit 1)
 				)
@@
 		(on_board yes)
 		(dnp no)
-		(property "Reference" "K1"
+		(property "Reference" "K9"
 			(at 134.874 32.258 0)
 			(effects
@@
 			(project "QMX-amp"
 				(path "/e63e39d7-6ac0-4ffd-8aa3-1841a4541b55/a2d04ef4-5ee1-49c1-8112-2f230613295c"
-					(reference "K1")
-					(unit 1)
-				)
+					(reference "K9")
+					(unit 1)
+				)
