File: amp-relay-ckt.kicad_sch (KiCad schematic)
At the start: 12 parts, among them Q2 MPS-751, Q5 BSS123, U1 LM7805_TO220

Commit message: v0.6 ERC passes.  I went over it with a fine tooth comb and corrected lots of little stuff.  Ron should review all the components I have to create very carefully.  In particular, MPS-751 symbol does not look correct.
Other:
- note removed: "+5V REG connects to bias pots. What is a 'bias pot' and where is it in the schematic?"
- note removed: "Are these the same K1 & K2 on p.2? YES How can I make K1 & K2 appear two different places yet be identical?"
- title: QMX Amp -> QMX+ Amp
- moved on the sheet: C17, C18, C19, C20, D10, D9, Q2, Q5, R2, R4, R7, U1

Commit message: v0.7 fixed MPS-751 and bifilar on FT50-43.  ERC passes
Connections:
- net +12V: now also Q2.1 (E); no longer Q2.3 (C)
- net at C18.1, U1.1 (VI): now also Q2.3 (C); no longer Q2.1 (E)
Changed lines of the file:
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@@
 		(title "QMX+ Amp")
 		(date "2024-08-13")
-		(rev "v0.6")
+		(rev "v0.7")
 		(company "WA7GIL")
 	)
@@
 	)
 	(junction
+		(at 139.7 102.87)
+		(diameter 0)
+		(color 0 0 0 0)
+	)
+	(junction
 		(at 124.46 76.2)
 		(diameter 0)
@@
 	)
 	(junction
-		(at 139.7 102.87)
+		(at 132.08 97.79)
 		(diameter 0)
 		(color 0 0 0 0)
@@
 	)
 	(junction
-		(at 132.08 97.79)
-		(diameter 0)
-		(color 0 0 0 0)
-	)
-	(junction
 		(at 160.02 102.87)
 		(diameter 0)
@@
 	(wire
 		(pts
+			(xy 139.7 91.44) (xy 139.7 92.71)
+		)
+		(stroke
+			(width 0)
+			(type default)
+		)
+	)
+	(wire
+		(pts
 			(xy 88.9 121.92) (xy 106.68 121.92)
 		)
@@
 		(pts
 			(xy 109.22 63.5) (xy 109.22 54.61)
-		)
-		(stroke
-			(width 0)
-			(type default)
-		)
-	)
-	(wire
-		(pts
-			(xy 139.7 91.44) (xy 139.7 92.71)
 		)
 		(stroke
@@
 		(lib_id "ZZZMyLibrary:MPS-751")
 		(at 137.16 97.79 0)
-		(unit 1)
-		(exclude_from_sim no)
-		(in_bom yes)
-		(on_board yes)
-		(dnp no)
-		(fields_autoplaced yes)
+		(mirror x)
+		(unit 1)
+		(exclude_from_sim no)
+		(in_bom yes)
+		(on_board yes)
+		(dnp no)
 		(property "Reference" "Q2"
-			(at 142.24 96.5199 0)
+			(at 142.24 99.0601 0)
 			(effects
 				(font
@@
 		)
 		(property "Value" "MPS-751"
-			(at 142.24 99.0599 0)
+			(at 142.24 96.5201 0)
 			(effects
 				(font
@@
 		)
 		(property "Footprint" ""
-			(at 142.24 95.25 0)
-			(effects
-				(font
+			(at 142.24 100.33 0)
+			(effects
+				(font

Commit message: ron came by and gave lots of feedback.  many notes on schematic for additional changes
Parts:
- C17, C18, C19, C20: footprint (none) -> ZZZMyLibrary:C_Disc_D11.0mm_W4.0mm_P5.00mm
- D10, D9: footprint (none) -> Diode_THT:D_DO-34_SOD68_P7.62mm_Horizontal
- Q2: footprint (none) -> Package_TO_SOT_THT:TO-92
- R2, R4, R7: footprint (none) -> Resistor_THT:R_Axial_DIN0309_L9.0mm_D3.2mm_P12.70mm_Horizontal
Changed lines of the file:
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@@
 			)
 		)
-		(property "Footprint" ""
+		(property "Footprint" "Resistor_THT:R_Axial_DIN0309_L9.0mm_D3.2mm_P12.70mm_Horizontal"
 			(at 104.902 125.73 90)
 			(effects
@@
 			)
 		)
-		(property "Footprint" ""
+		(property "Footprint" "Resistor_THT:R_Axial_DIN0309_L9.0mm_D3.2mm_P12.70mm_Horizontal"
 			(at 135.89 93.218 90)
 			(effects
@@
 			)
 		)
-		(property "Footprint" ""
+		(property "Footprint" "ZZZMyLibrary:C_Disc_D11.0mm_W4.0mm_P5.00mm"
 			(at 140.6652 110.49 0)
 			(effects
@@
 			)
 		)
-		(property "Footprint" ""
+		(property "Footprint" "Diode_THT:D_DO-34_SOD68_P7.62mm_Horizontal"
 			(at 193.04 67.31 0)
 			(effects
@@
 			)
 		)
-		(property "Footprint" ""
+		(property "Footprint" "ZZZMyLibrary:C_Disc_D11.0mm_W4.0mm_P5.00mm"
 			(at 89.8652 129.54 0)
 			(effects
@@
 			)
 		)
-		(property "Footprint" ""
+		(property "Footprint" "Diode_THT:D_DO-34_SOD68_P7.62mm_Horizontal"
 			(at 109.22 67.31 0)
 			(effects
@@
 			)
 		)
-		(property "Footprint" ""
+		(property "Footprint" "ZZZMyLibrary:C_Disc_D11.0mm_W4.0mm_P5.00mm"
 			(at 183.8452 110.49 0)
 			(effects
@@
 			)
 		)
-		(property "Footprint" ""
+		(property "Footprint" "Package_TO_SOT_THT:TO-92"
 			(at 142.24 100.33 0)
 			(effects
@@
 			)
 		)
-		(property "Footprint" ""
+		(property "Footprint" "Resistor_THT:R_Axial_DIN0309_L9.0mm_D3.2mm_P12.70mm_Horizontal"
 			(at 128.27 96.012 90)
 			(effects
@@
 			)
 		)
-		(property "Footprint" ""
+		(property "Footprint" "ZZZMyLibrary:C_Disc_D11.0mm_W4.0mm_P5.00mm"
 			(at 172.4152 71.12 0)
 			(effects

Commit message: expended to all 6 LPFs.  ERC pass.  Need to check component values on new LPF page
Parts:
- renumbered C20 to C17, C17 to C19, C19 to C20, Q2 to Q6, R7 to R5, R2 to R6, R4 to R7, U1 to U2
Changed lines of the file:
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@@
 		(dnp no)
 		(fields_autoplaced yes)
-		(property "Reference" "R7"
+		(property "Reference" "R5"
 			(at 109.22 124.4599 0)
 			(effects
@@
 			(project "QMX-amp"
 				(path "/e63e39d7-6ac0-4ffd-8aa3-1841a4541b55/6e8a5723-6162-4126-acdf-190058cf1f27"
-					(reference "R7")
+					(reference "R5")
 					(unit 1)
 				)
@@
 		(on_board yes)
 		(dnp no)
-		(property "Reference" "R4"
+		(property "Reference" "R7"
 			(at 135.89 85.09 90)
 			(effects
@@
 			(project "QMX-amp"
 				(path "/e63e39d7-6ac0-4ffd-8aa3-1841a4541b55/6e8a5723-6162-4126-acdf-190058cf1f27"
-					(reference "R4")
+					(reference "R7")
 					(unit 1)
 				)
@@
 		(dnp no)
 		(fields_autoplaced yes)
-		(property "Reference" "#PWR028"
+		(property "Reference" "#PWR034"
 			(at 106.68 135.89 0)
 			(effects
@@
 			(project "QMX-amp"
 				(path "/e63e39d7-6ac0-4ffd-8aa3-1841a4541b55/6e8a5723-6162-4126-acdf-190058cf1f27"
-					(reference "#PWR028")
+					(reference "#PWR034")
 					(unit 1)
 				)
@@
 		(dnp no)
 		(fields_autoplaced yes)
-		(property "Reference" "#FLG06"
+		(property "Reference" "#FLG03"
 			(at 160.02 100.965 0)
 			(effects
@@
 			(project ""
 				(path "/e63e39d7-6ac0-4ffd-8aa3-1841a4541b55/6e8a5723-6162-4126-acdf-190058cf1f27"
-					(reference "#FLG06")
+					(reference "#FLG03")
 					(unit 1)
 				)
@@
 		(dnp no)
 		(fields_autoplaced yes)
-		(property "Reference" "#PWR026"
+		(property "Reference" "#PWR038"
 			(at 173.99 116.84 0)
 			(effects
@@
 			(project "QMX-amp"
 				(path "/e63e39d7-6ac0-4ffd-8aa3-1841a4541b55/6e8a5723-6162-4126-acdf-190058cf1f27"
-					(reference "#PWR026")
+					(reference "#PWR038")
 					(unit 1)
 				)
@@
 		(dnp no)
 		(fields_autoplaced yes)
-		(property "Reference" "C20"
+		(property "Reference" "C17"
 			(at 92.71 123.5709 0)
 			(effects
@@
 			(project "QMX-amp"
 				(path "/e63e39d7-6ac0-4ffd-8aa3-1841a4541b55/6e8a5723-6162-4126-acdf-190058cf1f27"
-					(reference "C20")
+					(reference "C17")
 					(unit 1)
 				)
@@
 		(dnp no)
 		(fields_autoplaced yes)
-		(property "Reference" "#PWR029"
+		(property "Reference" "#PWR035"
 			(at 119.38 133.35 0)
 			(effects
@@
 			(project "QMX-amp"
 				(path "/e63e39d7-6ac0-4ffd-8aa3-1841a4541b55/6e8a5723-6162-4126-acdf-190058cf1f27"
-					(reference "#PWR029")
+					(reference "#PWR035")
 					(unit 1)
 				)
@@
 		(dnp no)
 		(fields_autoplaced yes)
-		(property "Reference" "U1"
+		(property "Reference" "U2"
 			(at 173.99 96.52 0)
 			(effects
@@
 			(project "QMX-amp"
 				(path "/e63e39d7-6ac0-4ffd-8aa3-1841a4541b55/6e8a5723-6162-4126-acdf-190058cf1f27"
-					(reference "U1")
+					(reference "U2")
 					(unit 1)
 				)
@@
 		(dnp no)
 		(fields_autoplaced yes)
-		(property "Reference" "#PWR024"
+		(property "Reference" "#PWR037"
 			(at 139.7 116.84 0)
 			(effects
@@
 			(project "QMX-amp"
 				(path "/e63e39d7-6ac0-4ffd-8aa3-1841a4541b55/6e8a5723-6162-4126-acdf-190058cf1f27"
-					(reference "#PWR024")
+					(reference "#PWR037")
 					(unit 1)
 				)
@@
 		(dnp no)
 		(fields_autoplaced yes)
-		(property "Reference" "#PWR032"
+		(property "Reference" "#PWR033"
 			(at 100.33 54.61 0)
 			(effects
@@
 			(project ""
 				(path "/e63e39d7-6ac0-4ffd-8aa3-1841a4541b55/6e8a5723-6162-4126-acdf-190058cf1f27"
-					(reference "#PWR032")
+					(reference "#PWR033")
 					(unit 1)
 				)
@@
 		(dnp no)
 		(fields_autoplaced yes)
-		(property "Reference" "#PWR025"
+		(property "Reference" "#PWR039"
 			(at 182.88 116.84 0)
 			(effects
@@
 			(project "QMX-amp"
 				(path "/e63e39d7-6ac0-4ffd-8aa3-1841a4541b55/6e8a5723-6162-4126-acdf-190058cf1f27"
-					(reference "#PWR025")
+					(reference "#PWR039")
 					(unit 1)
 				)
@@
 		(dnp no)
 		(fields_autoplaced yes)
-		(property "Reference" "#PWR027"
+		(property "Reference" "#PWR032"
 			(at 88.9 135.89 0)
 			(effects
@@
 			(project "QMX-amp"
 				(path "/e63e39d7-6ac0-4ffd-8aa3-1841a4541b55/6e8a5723-6162-4126-acdf-190058cf1f27"
-					(reference "#PWR027")
+					(reference "#PWR032")
 					(unit 1)
 				)
@@
 		(dnp no)
 		(fields_autoplaced yes)
-		(property "Reference" "C19"
+		(property "Reference" "C20"
 			(at 186.69 105.4099 0)
 			(effects
@@
 			(project "QMX-amp"
 				(path "/e63e39d7-6ac0-4ffd-8aa3-1841a4541b55/6e8a5723-6162-4126-acdf-190058cf1f27"
-					(reference "C19")
+					(reference "C20")
 					(unit 1)
 				)
@@
 		(on_board yes)
 		(dnp no)
-		(property "Reference" "Q2"
+		(property "Reference" "Q6"
 			(at 142.24 99.0601 0)
 			(effects
@@
 			(project ""
 				(path "/e63e39d7-6ac0-4ffd-8aa3-1841a4541b55/6e8a5723-6162-4126-acdf-190058cf1f27"
-					(reference "Q2")
+					(reference "Q6")
 					(unit 1)
 				)
@@
 		(on_board yes)
 		(dnp no)
-		(property "Reference" "R2"
+		(property "Reference" "R6"
 			(at 128.27 104.14 90)
 			(effects
@@
 			(project "QMX-amp"
 				(path "/e63e39d7-6ac0-4ffd-8aa3-1841a4541b55/6e8a5723-6162-4126-acdf-190058cf1f27"
-					(reference "R2")
+					(reference "R6")
 					(unit 1)
 				)
@@
 		(dnp no)
 		(fields_autoplaced yes)
-		(property "Reference" "#PWR031"
+		(property "Reference" "#PWR036"
 			(at 139.7 90.17 0)
 			(effects
@@
 			(project ""
 				(path "/e63e39d7-6ac0-4ffd-8aa3-1841a4541b55/6e8a5723-6162-4126-acdf-190058cf1f27"
-					(reference "#PWR031")
+					(reference "#PWR036")
 					(unit 1)
 				)
@@
 		(dnp no)
 		(fields_autoplaced yes)
-		(property "Reference" "C17"
+		(property "Reference" "C19"
 			(at 175.26 66.0399 0)
 			(effects
@@
 			(project "QMX-amp"
 				(path "/e63e39d7-6ac0-4ffd-8aa3-1841a4541b55/6e8a5723-6162-4126-acdf-190058cf1f27"
-					(reference "C17")
-					(unit 1)
-				)
+					(reference "C19")
+					(unit 1)
+				)
