File: amp.kicad_sch (KiCad schematic)
At the start: 17 parts, among them T1 BN-43-202, U3 RD16HHF1, U4 RD16HHF1

Commit message: checkpoint before I shrink width of capps  so things might fit PCB
Parts:
- RV1, RV2: footprint Resistor_THT:R_Axial_DIN0309_L9.0mm_D3.2mm_P12.70mm_Horizontal -> Potentiometer_THT:Potentiometer_Piher_PT-10-V05_Vertical
Connections:
- net K1-14 renamed K10-14
- net K2-14 renamed K9-14
Changed lines of the file:
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@@
 		(title "QMX+ Amp")
 		(date "2024-08-19")
-		(rev "v0.9")
+		(rev "v0.10")
 		(company "WA7GIL")
 	)
@@
 		)
 	)
-	(global_label "K2-14"
+	(global_label "K9-14"
 		(shape bidirectional)
 		(at 224.79 83.82 90)
@@
 		)
 	)
-	(global_label "K1-14"
+	(global_label "K10-14"
 		(shape bidirectional)
 		(at 80.01 83.82 180)
@@
 		)
 		(property "Intersheetrefs" "${INTERSHEET_REFS}"
-			(at 69.4428 83.82 0)
+			(at 68.2333 83.82 0)
 			(effects
 				(font
@@
 			)
 		)
-		(property "Footprint" "Resistor_THT:R_Axial_DIN0309_L9.0mm_D3.2mm_P12.70mm_Horizontal"
+		(property "Footprint" "Potentiometer_THT:Potentiometer_Piher_PT-10-V05_Vertical"
 			(at 144.78 64.77 0)
 			(effects
@@
 			)
 		)
-		(property "Footprint" "Resistor_THT:R_Axial_DIN0309_L9.0mm_D3.2mm_P12.70mm_Horizontal"
+		(property "Footprint" "Potentiometer_THT:Potentiometer_Piher_PT-10-V05_Vertical"
 			(at 147.32 113.03 0)
 			(effects

Commit message: v0.10 after slimming down capacitor width to 3mm so it *barely* fits.
Parts:
- C21, C22, C23, C24, C25: footprint ZZZMyLibrary:C_Disc_D11.0mm_W4.0mm_P5.00mm -> ZZZMyLibrary:C_Disc_D11.0mm_W3.0mm_P5.00mm
Changed lines of the file:
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@@
 			)
 		)
-		(property "Footprint" "ZZZMyLibrary:C_Disc_D11.0mm_W4.0mm_P5.00mm"
+		(property "Footprint" "ZZZMyLibrary:C_Disc_D11.0mm_W3.0mm_P5.00mm"
 			(at 182.88 97.4852 0)
 			(effects
@@
 			)
 		)
-		(property "Footprint" "ZZZMyLibrary:C_Disc_D11.0mm_W4.0mm_P5.00mm"
+		(property "Footprint" "ZZZMyLibrary:C_Disc_D11.0mm_W3.0mm_P5.00mm"
 			(at 135.89 112.0648 0)
 			(effects
@@
 			)
 		)
-		(property "Footprint" "ZZZMyLibrary:C_Disc_D11.0mm_W4.0mm_P5.00mm"
+		(property "Footprint" "ZZZMyLibrary:C_Disc_D11.0mm_W3.0mm_P5.00mm"
 			(at 135.89 67.6148 0)
 			(effects
@@
 			)
 		)
-		(property "Footprint" "ZZZMyLibrary:C_Disc_D11.0mm_W4.0mm_P5.00mm"
+		(property "Footprint" "ZZZMyLibrary:C_Disc_D11.0mm_W3.0mm_P5.00mm"
 			(at 135.89 82.8548 0)
 			(effects
@@
 			)
 		)
-		(property "Footprint" "ZZZMyLibrary:C_Disc_D11.0mm_W4.0mm_P5.00mm"
+		(property "Footprint" "ZZZMyLibrary:C_Disc_D11.0mm_W3.0mm_P5.00mm"
 			(at 135.89 94.9452 0)
 			(effects

Commit message: Ron helped moved all the parts into PCB
Parts:
- C21, C22, C23, C24: footprint ZZZMyLibrary:C_Disc_D11.0mm_W3.0mm_P5.00mm -> Resistor_SMD:R_0805_2012Metric_Pad1.20x1.40mm_HandSolder
- L10: footprint ZZZMyLibrary:BN-43-202-FLAT -> ZZZMyLibrary:BN-43-7051-FLAT
- R10, R8, R9: footprint Resistor_THT:R_Axial_DIN0309_L9.0mm_D3.2mm_P12.70mm_Horizontal -> Resistor_THT:R_Axial_DIN0207_L6.3mm_D2.5mm_P2.54mm_Vertical
- R11, R12: footprint Resistor_THT:R_Axial_DIN0309_L9.0mm_D3.2mm_P12.70mm_Horizontal -> Resistor_SMD:R_0805_2012Metric_Pad1.20x1.40mm_HandSolder
Changed lines of the file:
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@@
 			)
 		)
-		(property "Footprint" "Resistor_THT:R_Axial_DIN0309_L9.0mm_D3.2mm_P12.70mm_Horizontal"
+		(property "Footprint" "Resistor_THT:R_Axial_DIN0207_L6.3mm_D2.5mm_P2.54mm_Vertical"
 			(at 80.772 92.71 90)
 			(effects
@@
 			)
 		)
-		(property "Footprint" "ZZZMyLibrary:BN-43-202-FLAT"
+		(property "Footprint" "ZZZMyLibrary:BN-43-7051-FLAT"
 			(at 222.25 88.9 0)
 			(effects
@@
 			)
 		)
-		(property "Footprint" "ZZZMyLibrary:C_Disc_D11.0mm_W3.0mm_P5.00mm"
+		(property "Footprint" "Resistor_SMD:R_0805_2012Metric_Pad1.20x1.40mm_HandSolder"
 			(at 135.89 112.0648 0)
 			(effects
@@
 			)
 		)
-		(property "Footprint" "ZZZMyLibrary:C_Disc_D11.0mm_W3.0mm_P5.00mm"
+		(property "Footprint" "Resistor_SMD:R_0805_2012Metric_Pad1.20x1.40mm_HandSolder"
 			(at 135.89 67.6148 0)
 			(effects
@@
 			)
 		)
-		(property "Footprint" "ZZZMyLibrary:C_Disc_D11.0mm_W3.0mm_P5.00mm"
+		(property "Footprint" "Resistor_SMD:R_0805_2012Metric_Pad1.20x1.40mm_HandSolder"
 			(at 135.89 82.8548 0)
 			(effects
@@
 			)
 		)
-		(property "Footprint" "Resistor_THT:R_Axial_DIN0309_L9.0mm_D3.2mm_P12.70mm_Horizontal"
+		(property "Footprint" "Resistor_SMD:R_0805_2012Metric_Pad1.20x1.40mm_HandSolder"
 			(at 134.112 109.22 90)
 			(effects
@@
 			)
 		)
-		(property "Footprint" "Resistor_THT:R_Axial_DIN0309_L9.0mm_D3.2mm_P12.70mm_Horizontal"
+		(property "Footprint" "Resistor_SMD:R_0805_2012Metric_Pad1.20x1.40mm_HandSolder"
 			(at 134.112 72.39 90)
 			(effects
@@
 			)
 		)
-		(property "Footprint" "ZZZMyLibrary:C_Disc_D11.0mm_W3.0mm_P5.00mm"
+		(property "Footprint" "Resistor_SMD:R_0805_2012Metric_Pad1.20x1.40mm_HandSolder"
 			(at 135.89 94.9452 0)
 			(effects
@@
 			)
 		)
-		(property "Footprint" "Resistor_THT:R_Axial_DIN0309_L9.0mm_D3.2mm_P12.70mm_Horizontal"
+		(property "Footprint" "Resistor_THT:R_Axial_DIN0207_L6.3mm_D2.5mm_P2.54mm_Vertical"
 			(at 88.9 85.598 90)
 			(effects
@@
 			)
 		)
-		(property "Footprint" "Resistor_THT:R_Axial_DIN0309_L9.0mm_D3.2mm_P12.70mm_Horizontal"
+		(property "Footprint" "Resistor_THT:R_Axial_DIN0207_L6.3mm_D2.5mm_P2.54mm_Vertical"
 			(at 94.742 92.71 90)
 			(effects
